File: Eagle/drum_circuits.sch (EAGLE design)
At the start: 9 parts, among them J1 FTDI_BASICPTH, U1 ATMEGA328P_PDIP

Commit message: schematics
Parts:
- added C4: 0.1uF, SparkFun-Passives:CAPPTH
- added C5: 1uF, SparkFun-Passives:CAPPTH
- added C6: 10uF, SparkFun-Passives:CAPPTH
- added D1: (no value), SparkFun-LED:LTE-302
- added D2: (no value), SparkFun-DiscreteSemi:DIODEKIT2
- added FTDI: FTDI_BASICPTH, SparkFun-Connectors:FTDI_BASICPTH
- added ISP: AVR_SPI_PRG_6PTH, SparkFun-Connectors:AVR_SPI_PRG_6PTH
- added NRF: (no value), SparkFun-Connectors:M04X2
- added Q1: MOSFET-NCHANNELBS170, SparkFun-DiscreteSemi:MOSFET-NCHANNELBS170
- added R2, R3: 10k, SparkFun-Resistors:10KOHM-1/4W-1%(PTH)HORIZ-KIT
- added SOLNOID: (no value), SparkFun-Connectors:M02PTH
- C1, C2: value 10pf -> 22pF
- C3: value (none) -> 0.1uF
- J1: value FTDI_BASICPTH -> (none); device SparkFun-Connectors:FTDI_BASICPTH -> SparkFun-Connectors:M03PTH
- renumbered U2 to VREG3.3V
Connections:
- removed net N$2: U1.PD2(INT0)
- new net CE: NRF.3, U1.PB0(ICP)
- new net CSN: NRF.4, U1.PB2(SS/OC1B)
- new net DRAIN: D2.A, Q1.G, SOLNOID.2
- new net DTR: C4.1, FTDI.1
- new net LED: R2.2, U1.PD3(INT1)
- new net MIC: J1.3, U1.PC0(ADC0)
- new net MISO: ISP.1, NRF.7, U1.PB4(MISO)
- new net MOSI: ISP.4, NRF.6, U1.PB3(MOSI/OC2)
- new net RST: C4.2, ISP.5, R1.1, S1.3, S1.4, U1.PC6(/RESET)
- new net SCK: ISP.3, NRF.5, U1.PB5(SCK)
- new net SOLENOID: Q1.D, R3.2, U1.PD4(XCK/T0)
- net 3.3V: now also FTDI.4, ISP.2, J1.1, NRF.2, R1.2; no longer J1.4
- net GND: now also C5.2, C6.2, D1.C, FTDI.6, ISP.6, J1.2, NRF.1, Q1.S, R3.1; no longer J1.6
- net N$1: now also D1.A, R2.1; no longer R1.1, S1.3, S1.4, U1.PC6(/RESET)
- net RX: now also FTDI.2; no longer J1.2
- net TX: now also FTDI.3; no longer J1.3
- net VCC: now also C5.1, C6.1, D2.C, SOLNOID.1; no longer R1.2
- net XTAL1: now also U1.PB6(XTAL1/TOSC1)
- net XTAL2: now also U1.PB7(XTAL2/TOSC2)
