File: circuits/drum_circuits.sch (EAGLE design)
At the start: 39 parts, among them U1 OPA344, U2 ATMEGA328P_TQFP, U3 ADMP401

Commit message: overwriting board & schematic from 5d2ad6c18a5f5ec5e8afae34b5d28b62efabe567
Parts:
- removed 5VREG: MIC5225-5v, adafruit:LP298XS
- removed C10: 1uF, fab:CAP-UNPOLARIZEDFAB
- removed C11: 100pF, fab:CAP-UNPOLARIZEDFAB
- removed C12, C13: 0.1uF, fab:CAP-UNPOLARIZEDFAB
- removed C6, C9: 10uF, talkingdrums:POLCAP-PANASONIC-SMD-B01
- removed NRFCAP: 33uF, talkingdrums:POLCAP-PANASONIC-SMD-C
- removed R5: 500, fab:RES-US1206FAB
- removed R6: 1.5K, fab:RES-US1206FAB
- removed R7, R8: 10k, fab:RES-US1206FAB
- removed R9: 100k, fab:RES-US1206FAB
- removed SC1, SC2: (no value), adafruit:DIODE_SOD-123FL
- removed U1: OPA344, SparkFun-AnalogIC:OPA344
- removed U3: ADMP401, SparkFun-Sensors:ADMP401
- added C7: 10uF, talkingdrums:POLCAP-PANASONIC-SMD-B01
- added MIC: (no value), SparkFun-Connectors:M03PTH
- added U$3: RECTIFIER, talkingdrums:RECTIFIER
- added VREG5.5V: 7805, fab:REGULATORSOT23
- C8: value 4.7uF -> 10uF; device fab:CAP-UNPOLARIZEDFAB -> talkingdrums:POLCAP-PANASONIC-SMD-B01
- D2: value LEDFAB1206 -> RECTIFIER; device fab:LEDFAB1206 -> talkingdrums:RECTIFIER
Connections:
- net N$10 renamed LED
- net N$11 renamed GATE
- removed net N$6: D2.A, R5.2
- removed net N$7: C8.2, R6.2
- removed net N$8: C10.2, C11.1, R6.1, R7.2, R8.2, R9.2, U1.+IN, U1.-IN
- removed net N$9: C13.2, U2.AREF
- removed net VBUS: ISP.2, SC1.A, U$1.VCC
- net 3.3V: no longer C12.2, R7.1, U1.V+, U3.VDD
- net 5V: now also C8.+, ISP.2, MIC.1, U$1.VCC, U2.AREF, VREG5.5V.OUT; no longer 5VREG.VOUT, C9.+, R5.1, SC1.C
- net DRAIN: now also U$3.1; no longer SC2.A
- net GND: now also C7.-, C8.-, MIC.2, VREG5.5V.GND; no longer 5VREG.GND, C10.1, C12.1, C13.1, C6.-, C9.-, D2.C, R8.1, U$1.CTS, U1.V-, U3.GND@2, U3.GND@4, U3.GND@6
- net MIC: now also MIC.3; no longer C11.2, R9.1, U1.OUT
- net N$4: now also C7.+, D2.2, VREG5.5V.IN; no longer C8.1, U3.OUT
- net VCC: now also D2.1, U$3.2; no longer 5VREG.EN, 5VREG.VIN, C6.+, SC2.C
Other:
- note added: "NEW REGULATOR"
- note removed: "JUMPERS"
- note removed: "MIC"
- note removed: "MICROCONTROLLER"
- note removed: "POWER"
- note removed: "SOLENOID"
- moved on the sheet: BAT, C1, C2, C3, C4, C5, CRYSTAL, D1, ISP, Q2, R1, R2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

Commit message: schematics and parts_list
Parts:
- removed C7: 10uF, talkingdrums:POLCAP-PANASONIC-SMD-B01
- removed MIC: (no value), SparkFun-Connectors:M03PTH
- removed U$3: RECTIFIER, talkingdrums:RECTIFIER
- removed VREG5.5V: 7805, fab:REGULATORSOT23
- added C10: 1uF, fab:CAP-UNPOLARIZEDFAB
- added C11: 100pF, fab:CAP-UNPOLARIZEDFAB
- added C12, C13: 0.1uF, fab:CAP-UNPOLARIZEDFAB
- added C6, C9: 10uF, talkingdrums:POLCAP-PANASONIC-SMD-B01
- added IC2: MIC5225-5v, adafruit:LP298XS
- added R5: 500, fab:RES-US1206FAB
- added R6: 1.5K, fab:RES-US1206FAB
- added R7, R8: 10k, fab:RES-US1206FAB
- added R9: 100k, fab:RES-US1206FAB
- added SCHOTTKY, SCHOTTKY1: (no value), adafruit:DIODE_SOD-123FL
- added U$4: 33uF, talkingdrums:POLCAP-PANASONIC-SMD-C
- added U1: OPA344, SparkFun-AnalogIC:OPA344
- added U3: ADMP401, SparkFun-Sensors:ADMP401
- C8: value 10uF -> 4.7uF; device talkingdrums:POLCAP-PANASONIC-SMD-B01 -> fab:CAP-UNPOLARIZEDFAB
- D2: value RECTIFIER -> LEDFAB1206; device talkingdrums:RECTIFIER -> fab:LEDFAB1206
Connections:
- net GATE renamed N$11
- net LED renamed N$10
- new net N$12: U$2.VCC
- new net N$6: D2.A, R5.2
- new net N$7: C8.2, R6.2
- new net N$8: C10.2, C11.1, R6.1, R7.2, R8.2, R9.2, U1.+IN, U1.-IN
- new net N$9: C13.2, U2.AREF
- new net VBUS: ISP.2, SCHOTTKY.A, U$1.VCC
- net 3.3V: now also C12.2, R7.1, U1.V+, U3.VDD; no longer U$2.VCC
- net 5V: now also C9.+, IC2.VOUT, R5.1, SCHOTTKY.C; no longer C8.+, ISP.2, MIC.1, U$1.VCC, U2.AREF, VREG5.5V.OUT
- net DRAIN: now also SCHOTTKY1.A; no longer U$3.1
- net GND: now also C10.1, C12.1, C13.1, C6.-, C9.-, D2.C, IC2.GND, R8.1, U$1.CTS, U1.V-, U3.GND@2, U3.GND@4, U3.GND@6; no longer C7.-, C8.-, MIC.2, VREG5.5V.GND
- net MIC: now also C11.2, R9.1, U1.OUT; no longer MIC.3
- net N$4: now also C8.1, U3.OUT; no longer C7.+, D2.2, VREG5.5V.IN
- net VCC: now also C6.+, IC2.EN, IC2.VIN, SCHOTTKY1.C; no longer D2.1, U$3.2
Other:
- note added: "JUMPERS"
- note added: "MIC"
- note added: "MICROCONTROLLER"
- note added: "POWER"
- note added: "SOLENOID"
- note removed: "NEW REGULATOR"
- moved on the sheet: BAT, C1, C2, C3, C4, C5, CRYSTAL, D1, ISP, Q2, R1, R2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

Commit message: categorize parts
Parts:
- renumbered IC2 to 5VREG, SCHOTTKY to SC1, SCHOTTKY1 to SC2, U$4 to NRFCAP
Connections:
- removed net N$12: U$2.VCC
- net 3.3V: now also U$2.VCC
Changed lines of the file:
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@@
 <part name="S1" library="fab" deviceset="6MM_SWITCH" device="6MM_SWITCH"/>
 <part name="U2" library="SparkFun-DigitalIC" deviceset="ATMEGA328P_TQFP" device="" value="ATMEGA328P_TQFP"/>
-<part name="IC2" library="adafruit" deviceset="LP298X" device="S" value="MIC5225-5v"/>
+<part name="5VREG" library="adafruit" deviceset="LP298X" device="S" value="MIC5225-5v"/>
 <part name="C6" library="talkingdrums" deviceset="POLCAP-PANASONIC-SMD-B" device="01" value="10uF"/>
 <part name="C9" library="talkingdrums" deviceset="POLCAP-PANASONIC-SMD-B" device="01" value="10uF"/>
 <part name="R5" library="fab" deviceset="RES-US" device="1206FAB" value="500"/>
-<part name="SCHOTTKY" library="adafruit" deviceset="DIODE" device="_SOD-123FL"/>
+<part name="SC1" library="adafruit" deviceset="DIODE" device="_SOD-123FL"/>
 <part name="D2" library="fab" deviceset="LED" device="FAB1206"/>
 <part name="U3" library="SparkFun-Sensors" deviceset="ADMP401" device=""/>
@@
 <part name="C12" library="fab" deviceset="CAP-UNPOLARIZED" device="FAB" value="0.1uF"/>
 <part name="C13" library="fab" deviceset="CAP-UNPOLARIZED" device="FAB" value="0.1uF"/>
-<part name="U$4" library="talkingdrums" deviceset="POLCAP-PANASONIC-SMD-C" device="" value="33uF"/>
-<part name="SCHOTTKY1" library="adafruit" deviceset="DIODE" device="_SOD-123FL"/>
+<part name="NRFCAP" library="talkingdrums" deviceset="POLCAP-PANASONIC-SMD-C" device="" value="33uF"/>
+<part name="SC2" library="adafruit" deviceset="DIODE" device="_SOD-123FL"/>
 </parts>
 <sheets>
@@
 <instance part="S1" gate="2" x="48.26" y="-38.1"/>
 <instance part="U2" gate="U$1" x="109.22" y="-63.5"/>
-<instance part="IC2" gate="G$1" x="53.34" y="-454.66" rot="R270"/>
+<instance part="5VREG" gate="G$1" x="53.34" y="-454.66" rot="R270"/>
 <instance part="C6" gate="G$1" x="15.24" y="-457.2" rot="R90"/>
 <instance part="C9" gate="G$1" x="88.9" y="-459.74" rot="R90"/>
 <instance part="R5" gate="G$1" x="76.2" y="-459.74" rot="R270"/>
-<instance part="SCHOTTKY" gate="G$1" x="68.58" y="-434.34" rot="R270"/>
+<instance part="SC1" gate="G$1" x="68.58" y="-434.34" rot="R270"/>
 <instance part="D2" gate="G$1" x="76.2" y="-472.44"/>
 <instance part="U3" gate="G$1" x="30.48" y="-340.36"/>
@@
 <instance part="C12" gate="&gt;NAME" x="101.6" y="-360.68" rot="R90"/>
 <instance part="C13" gate="&gt;NAME" x="71.12" y="-48.26"/>
-<instance part="U$4" gate="G$1" x="152.4" y="-269.24" rot="R180"/>
-<instance part="SCHOTTKY1" gate="G$1" x="137.16" y="-170.18"/>
+<instance part="NRFCAP" gate="G$1" x="152.4" y="-269.24" rot="R180"/>
+<instance part="SC2" gate="G$1" x="137.16" y="-170.18"/>
 </instances>
 <busses>
@@
 </segment>
 <segment>
-<pinref part="IC2" gate="G$1" pin="VOUT"/>
+<pinref part="5VREG" gate="G$1" pin="VOUT"/>
 <wire x1="63.5" y1="-449.58" x2="68.58" y2="-449.58" width="0.1524" layer="91"/>
 <wire x1="68.58" y1="-449.58" x2="76.2" y2="-449.58" width="0.1524" layer="91"/>
@@
 <wire x1="76.2" y1="-454.66" x2="76.2" y2="-449.58" width="0.1524" layer="91"/>
 <junction x="76.2" y="-449.58"/>
-<pinref part="SCHOTTKY" gate="G$1" pin="C"/>
+<pinref part="SC1" gate="G$1" pin="C"/>
 <wire x1="68.58" y1="-436.88" x2="68.58" y2="-449.58" width="0.1524" layer="91"/>
 <junction x="68.58" y="-449.58"/>
@@
 <wire x1="170.18" y1="-269.24" x2="170.18" y2="-254" width="0.1524" layer="91"/>
 <junction x="170.18" y="-254"/>
+<label x="170.18" y="-266.7" size="1.778" layer="95"/>
 </segment>
 <segment>
@@
 <segment>
 <wire x1="27.94" y1="-480.06" x2="27.94" y2="-454.66" width="0.1524" layer="91"/>
-<pinref part="IC2" gate="G$1" pin="GND"/>
+<pinref part="5VREG" gate="G$1" pin="GND"/>
 <wire x1="27.94" y1="-454.66" x2="38.1" y2="-454.66" width="0.1524" layer="91"/>
 <label x="25.4" y="-482.6" size="1.778" layer="95"/>
@@
 </segment>
 <segment>
-<pinref part="IC2" gate="G$1" pin="VIN"/>
+<pinref part="5VREG" gate="G$1" pin="VIN"/>
 <wire x1="38.1" y1="-449.58" x2="35.56" y2="-449.58" width="0.1524" layer="91"/>
 <wire x1="35.56" y1="-449.58" x2="15.24" y2="-449.58" width="0.1524" layer="91"/>
@@
 <wire x1="7.62" y1="-449.58" x2="7.62" y2="-439.42" width="0.1524" layer="91"/>
 <label x="5.08" y="-439.42" size="1.778" layer="95"/>
-<pinref part="IC2" gate="G$1" pin="EN"/>
+<pinref part="5VREG" gate="G$1" pin="EN"/>
 <wire x1="38.1" y1="-459.74" x2="35.56" y2="-459.74" width="0.1524" layer="91"/>
 <wire x1="35.56" y1="-459.74" x2="35.56" y2="-449.58" width="0.1524" layer="91"/>
@@
 </segment>
 <segment>
-<pinref part="SCHOTTKY1" gate="G$1" pin="C"/>
+<pinref part="SC2" gate="G$1" pin="C"/>
 <wire x1="139.7" y1="-170.18" x2="147.32" y2="-170.18" width="0.1524" layer="91"/>
 <label x="149.86" y="-170.18" size="1.778" layer="95"/>
@@
 </segment>
 <segment>
-<pinref part="SCHOTTKY1" gate="G$1" pin="A"/>
+<pinref part="SC2" gate="G$1" pin="A"/>
 <wire x1="134.62" y1="-170.18" x2="124.46" y2="-170.18" width="0.1524" layer="91"/>
 <label x="121.92" y="-170.18" size="1.778" layer="95"/>
@@
 <wire x1="101.6" y1="-358.14" x2="101.6" y2="-353.06" width="0.1524" layer="91"/>
 <label x="99.06" y="-350.52" size="1.778" layer="95"/>
+</segment>
+<segment>
+<pinref part="U$2" gate="G$1" pin="VCC"/>
+<wire x1="139.7" y1="-254" x2="134.62" y2="-254" width="0.1524" layer="91"/>
+<label x="134.62" y="-254" size="1.778" layer="95"/>
+<wire x1="149.86" y1="-269.24" x2="139.7" y2="-269.24" width="0.1524" layer="91"/>
+<wire x1="139.7" y1="-269.24" x2="139.7" y2="-254" width="0.1524" layer="91"/>
+<junction x="139.7" y="-254"/>
+<label x="137.16" y="-266.7" size="1.778" layer="95"/>
 </segment>
 </net>
@@
 <net name="VBUS" class="0">
 <segment>
-<pinref part="SCHOTTKY" gate="G$1" pin="A"/>
+<pinref part="SC1" gate="G$1" pin="A"/>
 <wire x1="68.58" y1="-431.8" x2="68.58" y2="-426.72" width="0.1524" layer="91"/>
 <label x="68.58" y="-426.72" size="1.778" layer="95"/>
@@
 </segment>
 </net>
-<net name="N$12" class="0">
-<segment>
-<pinref part="U$2" gate="G$1" pin="VCC"/>
-<wire x1="139.7" y1="-254" x2="137.16" y2="-254" width="0.1524" layer="91"/>
-<label x="134.62" y="-254" size="1.778" layer="95"/>
-<wire x1="137.16" y1="-254" x2="134.62" y2="-254" width="0.1524" layer="91"/>
-<wire x1="149.86" y1="-269.24" x2="137.16" y2="-269.24" width="0.1524" layer="91"/>
-<wire x1="137.16" y1="-269.24" x2="137.16" y2="-254" width="0.1524" layer="91"/>
-<junction x="137.16" y="-254"/>
-</segment>
-</net>
