File: circuits/drum_circuits.brd (EAGLE design)
At the start: 33 x 46.1 mm, 26 parts, among them U2 ATMEGA328P_TQFP

Commit message: schematics and parts_list
Parts:
- removed C7: 10uF, talkingdrums:PANASONIC-CAP-SMD-B
- removed MIC: (no value), SparkFun-Connectors:1X03
- removed U$3: RECTIFIER, talkingdrums:RECTIFIER
- removed VREG5.5V: 7805, fab:SOT23
- added C10: 1uF, fab:C1206FAB
- added C11: 100pF, fab:C1206FAB
- added C12, C13: 0.1uF, fab:C1206FAB
- added C6, C9: 10uF, talkingdrums:PANASONIC-CAP-SMD-B
- added IC2: MIC5225-5v, adafruit:SOT23-5L
- added R5: 500, fab:R1206FAB
- added R6: 1.5K, fab:R1206FAB
- added R7, R8: 10k, fab:R1206FAB
- added R9: 100k, fab:R1206FAB
- added SCHOTTKY, SCHOTTKY1: (no value), adafruit:SOD-123FL
- added U$4: 33uF, talkingdrums:PANASONIC-CAP-SMD-C
- added U1: OPA344, SparkFun-AnalogIC:SOT23-5
- added U3: ADMP401, SparkFun-Sensors:ADMP401
- C8: value 10uF -> 4.7uF; device talkingdrums:PANASONIC-CAP-SMD-B -> fab:C1206FAB
- D2: value RECTIFIER -> LEDFAB1206; device talkingdrums:RECTIFIER -> fab:LED1206FAB
- moved C8 100.9 mm to (-7.90, -53.1), turned to 0 degrees
- moved D2 77.8 mm to (0.00, -39.8), turned to 0 degrees
Connections:
- net GATE renamed N$11
- net LED renamed N$10
- new net N$12: U$2.2
- new net N$6: D2.1, R5.2
- new net N$7: C8.2, R6.2
- new net N$8: C10.2, C11.1, R6.1, R7.2, R8.2, R9.2, U1.3, U1.4
- new net N$9: C13.2, U2.20
- new net VBUS: ISP.2, SCHOTTKY.A, U$1.3
- net 3.3V: now also C12.2, R7.1, U1.5, U3.5; no longer U$2.2
- net 5V: now also C9.POS, IC2.5, R5.1, SCHOTTKY.C; no longer C8.POS, ISP.2, MIC.1, U$1.3, U2.20, VREG5.5V.1
- net DRAIN: now also SCHOTTKY1.A; no longer U$3.1
- net GND: now also C10.1, C12.1, C13.1, C6.NEG, C9.NEG, D2.2, IC2.2, R8.1, U$1.2, U1.2, U3.2, U3.4, U3.6; no longer C7.NEG, C8.NEG, MIC.2, VREG5.5V.3
- net MIC: now also C11.2, R9.1, U1.1; no longer MIC.3
- net N$4: now also C8.1, U3.1; no longer C7.POS, D2.2, VREG5.5V.2
- net VCC: now also C6.POS, IC2.1, IC2.3, SCHOTTKY1.C; no longer D2.1, U$3.2
Routing:
- net 5V: track 121.8 -> 83.3 mm
- net GND: track 223.6 -> 192.3 mm
- net N$4: track 13.0 -> 0.00 mm
- net N$11: track 8.26 -> 0.00 mm
- net N$10: track 5.40 -> 0.00 mm
- net 3.3V: track 3.17 -> 0.00 mm
- net N$12: track 0.00 -> 2.94 mm
- net VCC: track 33.1 -> 32.6 mm

Commit message: categorize parts
Parts:
- removed IC2: MIC5225-5v, adafruit:SOT23-5L
- removed SCHOTTKY, SCHOTTKY1: (no value), adafruit:SOD-123FL
- removed U$4: 33uF, talkingdrums:PANASONIC-CAP-SMD-C
- added 5VREG: MIC5225-5v, adafruit:SOT23-5L
- added NRFCAP: 33uF, talkingdrums:PANASONIC-CAP-SMD-C
- added SC1, SC2: (no value), adafruit:SOD-123FL
- moved C11 133.4 mm to (65.7, 25.2), turned to 180 degrees
- moved C12 127.4 mm to (71.6, 8.00)
- moved C13 127.2 mm to (17.9, 27.5)
- moved R9 124.4 mm to (65.7, 19.7)
- moved R7 106.7 mm to (59.8, 18.4), turned to 180 degrees
- moved C10 103.1 mm to (57.2, 4.90), turned to 90 degrees
- moved R8 102.1 mm to (63.6, 3.30)
- moved U1 99.6 mm to (68.4, 14.8), turned to 270 degrees
- moved R6 99.4 mm to (61.1, 13.0), turned to 90 degrees
- moved C8 92.4 mm to (57.5, 12.2), turned to 90 degrees
- moved U3 91.5 mm to (71.0, 4.20), turned to 270 degrees
- moved D2 74.8 mm to (30.6, 28.5), turned to 90 degrees
- moved R5 68.2 mm to (30.3, 34.9), turned to 90 degrees
- moved C9 61.7 mm to (24.6, 36.0), turned to 180 degrees
- moved U$2 53.5 mm to (58.2, 32.1), flipped to the top, turned to 270 degrees
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Connections:
- removed net N$12: U$2.2
- net 3.3V: now also U$2.2
- net 5V: now also 5VREG.5, SC1.C; no longer IC2.5, SCHOTTKY.C
- net DRAIN: now also SC2.A; no longer SCHOTTKY1.A
- net GND: now also 5VREG.2; no longer IC2.2
- net VBUS: now also SC1.A; no longer SCHOTTKY.A
- net VCC: now also 5VREG.1, 5VREG.3, SC2.C; no longer IC2.1, IC2.3, SCHOTTKY1.C
Routing:
- net GND: track 192.3 -> 0.00 mm, vias 1 -> 0
- net 5V: track 83.3 -> 0.00 mm, vias 3 -> 0
- net RST: track 77.8 -> 0.00 mm, vias 1 -> 0
- net MISO: track 66.5 -> 0.00 mm, vias 3 -> 0
- net MOSI: track 46.9 -> 0.00 mm, vias 1 -> 0
- net SCK: track 43.4 -> 0.00 mm, vias 1 -> 0
- net RX: track 33.3 -> 0.00 mm
- net VCC: track 32.6 -> 0.00 mm
- net TX: track 24.1 -> 0.00 mm
- net GATE_DO: track 19.5 -> 0.00 mm
- net DRAIN: track 14.0 -> 0.00 mm
- net CE: track 13.6 -> 0.00 mm, vias 1 -> 0
- net DTR: track 12.5 -> 0.00 mm
- net CSN: track 11.4 -> 0.00 mm, vias 1 -> 0
- net XTAL2: track 11.2 -> 0.00 mm, vias 1 -> 0
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Other:
- board size 33 x 46.1 mm -> 79.9 x 51.2 mm
- board text removed: "+"
- board text removed: "-"
- board text removed: "G"

Commit message: overwriting board & schematic from 5d2ad6c18a5f5ec5e8afae34b5d28b62efabe567
Parts:
- removed 5VREG: MIC5225-5v, adafruit:SOT23-5L
- removed C10: 1uF, fab:C1206FAB
- removed C11: 100pF, fab:C1206FAB
- removed C12, C13: 0.1uF, fab:C1206FAB
- removed C6, C9: 10uF, talkingdrums:PANASONIC-CAP-SMD-B
- removed NRFCAP: 33uF, talkingdrums:PANASONIC-CAP-SMD-C
- removed R5: 500, fab:R1206FAB
- removed R6: 1.5K, fab:R1206FAB
- removed R7, R8: 10k, fab:R1206FAB
- removed R9: 100k, fab:R1206FAB
- removed SC1, SC2: (no value), adafruit:SOD-123FL
- removed U1: OPA344, SparkFun-AnalogIC:SOT23-5
- removed U3: ADMP401, SparkFun-Sensors:ADMP401
- added C7: 10uF, talkingdrums:PANASONIC-CAP-SMD-B
- added MIC: (no value), SparkFun-Connectors:1X03
- added U$3: RECTIFIER, talkingdrums:RECTIFIER
- added VREG5.5V: 7805, fab:SOT23
- C8: value 4.7uF -> 10uF; device fab:C1206FAB -> talkingdrums:PANASONIC-CAP-SMD-B
- D2: value LEDFAB1206 -> RECTIFIER; device fab:LED1206FAB -> talkingdrums:RECTIFIER
- moved U$2 53.5 mm to (5.80, 21.4), flipped to the bottom, turned to 0 degrees
- moved C8 46.0 mm to (23.2, 42.9), turned to 180 degrees
- moved VREG3.3 44.6 mm to (10.4, 17.4), flipped to the bottom
- moved C3 34.0 mm to (5.35, 32.7), flipped to the bottom, turned to 0 degrees
- moved BAT 23.0 mm to (28.7, 34.9)
- moved C4 21.4 mm to (27.4, 27.1), turned to 180 degrees
- moved D1 21.4 mm to (6.85, 2.69), turned to 180 degrees
- moved ISP 20.7 mm to (27.1, 14.8), flipped to the bottom, turned to 270 degrees
- moved R4 19.6 mm to (10.6, 26.0), turned to 0 degrees
- moved C5 17.5 mm to (18.0, 29.4), turned to 180 degrees
- moved S1 17.0 mm to (19.7, 22.3)
- moved U2 15.7 mm to (11.6, 10.5), turned to 180 degrees
- moved R1 14.2 mm to (27.3, 21.5), turned to 180 degrees
- moved R2 13.1 mm to (13.5, 2.68), turned to 0 degrees
- moved D2 12.4 mm to (20.2, 35.3), turned to 180 degrees
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Connections:
- net N$10 renamed LED
- net N$11 renamed GATE
- removed net N$6: D2.1, R5.2
- removed net N$7: C8.2, R6.2
- removed net N$8: C10.2, C11.1, R6.1, R7.2, R8.2, R9.2, U1.3, U1.4
- removed net N$9: C13.2, U2.20
- removed net VBUS: ISP.2, SC1.A, U$1.3
- net 3.3V: no longer C12.2, R7.1, U1.5, U3.5
- net 5V: now also C8.POS, ISP.2, MIC.1, U$1.3, U2.20, VREG5.5V.1; no longer 5VREG.5, C9.POS, R5.1, SC1.C
- net DRAIN: now also U$3.1; no longer SC2.A
- net GND: now also C7.NEG, C8.NEG, MIC.2, VREG5.5V.3; no longer 5VREG.2, C10.1, C12.1, C13.1, C6.NEG, C9.NEG, D2.2, R8.1, U$1.2, U1.2, U3.2, U3.4, U3.6
- net MIC: now also MIC.3; no longer C11.2, R9.1, U1.1
- net N$4: now also C7.POS, D2.2, VREG5.5V.2; no longer C8.1, U3.1
- net VCC: now also D2.1, U$3.2; no longer 5VREG.1, 5VREG.3, C6.POS, SC2.C
Routing:
- net GND: track 0.00 -> 223.6 mm, vias 0 -> 1
- net 5V: track 0.00 -> 121.8 mm, vias 0 -> 3
- net RST: track 0.00 -> 77.8 mm, vias 0 -> 1
- net MISO: track 0.00 -> 66.5 mm, vias 0 -> 3
- net MOSI: track 0.00 -> 46.9 mm, vias 0 -> 1
- net SCK: track 0.00 -> 43.4 mm, vias 0 -> 1
- net RX: track 0.00 -> 33.3 mm
- net VCC: track 0.00 -> 33.1 mm
- net TX: track 0.00 -> 24.1 mm
- net GATE_DO: track 0.00 -> 19.5 mm
- net DRAIN: track 0.00 -> 14.1 mm
- net CE: track 0.00 -> 13.6 mm, vias 0 -> 1
- net N$4: track 0.00 -> 13.0 mm
- net DTR: track 0.00 -> 12.5 mm
- net CSN: track 0.00 -> 11.4 mm, vias 0 -> 1
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Other:
- board size 79.9 x 51.2 mm -> 33 x 46.1 mm
- board text added: "+"
- board text added: "-"
- board text added: "G"
