File: circuits/2017-09-15_drum_circuits.sch (EAGLE design)
At the start: 30 parts, among them IC2 MIC5225-5v, U2 ATMEGA328P_TQFP

Commit message: clean
Parts:
- removed Q2: (no value), fab:NMOSFETSOT23
- removed R3: 10k, fab:RES-US1206FAB
- removed R4: 100, fab:RES-US1206FAB
- removed SCHOTTKY1: (no value), adafruit:DIODE_SOD-123FL
- added H_BRIDGE_INA, H_BRIDGE_OUT: (no value), pinhead-2:PINHD-1X05_2.54-SMD
- added PC, PM, PS: (no value), adafruit:TRIMPOTTC33X
- added U$3: SWITCH_SPDT, SparkFun-Electromechanical:SWITCH_SPDT
Connections:
- removed net DRAIN: Q2.D, SCHOTTKY1.A, SOLNOID.2
- removed net GATE_DO: R3.2, R4.1, U2.PD5(T1)
- removed net N$11: Q2.G, R4.2
- new net BAT_IN: BAT.2, U$3.P
- new net ENABLE: H_BRIDGE_INA.3, U2.PD4(XCK/T0)
- new net OUT: U$3.S
- new net PHASE: H_BRIDGE_INA.4, U2.PD5(T1)
- new net PM: PM.S, U2.PC1(ADC1)
- new net POT_C: PC.S, U2.PC3(ADC3)
- new net POT_S: PS.S, U2.PC2(ADC2)
- new net SLEEP: H_BRIDGE_INA.5, U2.PD6(AIN0)
- new net SOL_1: H_BRIDGE_OUT.4, SOLNOID.1
- new net SOL_2: H_BRIDGE_OUT.3, SOLNOID.2
- new net VM: H_BRIDGE_OUT.5
- net 3.3V: now also MIC.1
- net 5V: now also H_BRIDGE_INA.2, PC.A, PM.A, PS.A; no longer MIC.1
- net GND: now also H_BRIDGE_INA.1, H_BRIDGE_OUT.1, PC.E, PM.E, PS.E; no longer Q2.S, R3.1
- net VCC: now also H_BRIDGE_OUT.2, U$3.O; no longer BAT.2, SCHOTTKY1.C, SOLNOID.1
Other:
- note added: "CONTROLLERS"
- note removed: "mosfet"
- note removed: "pulldwn"
- note removed: "source"
